Commit message: Added new model with working husky

File: models/hdt_michigan_description/urdf/gazebo_utilities.xacro (robot description, xacro)
@@ -65,6 +65,6 @@
                 <!--  This must be the same as the root frame of the robot you're using -->
                 <frameId>${root_frame_id}</frameId>
-                <excludedModels>collision_sphere</excludedModels>
-                <scalePrimitivesFactor>1.1</scalePrimitivesFactor>
+                <excludedModels>collision_sphere my_ground_plane</excludedModels>
+                <scalePrimitivesFactor>1.0</scalePrimitivesFactor>
             </plugin>
         </gazebo>

File: models/hdt_michigan_description/urdf/hdt_michigan_no_husky.xacro (robot description, xacro)
@@ -1,15 +1,4 @@
 <?xml version="1.0"?>
-<robot name="hdt_michigan" xmlns:xacro="http://www.ros.org/wiki/xacro">
-    <xacro:macro name="collision_visual" params="name *origin *geometry *material">
-        <collision name="${name}_collision">
-            <xacro:insert_block name="origin"/>
-            <xacro:insert_block name="geometry"/>
-        </collision>
-        <visual name="${name}_visual">
-            <xacro:insert_block name="origin"/>
-            <xacro:insert_block name="geometry"/>
-            <xacro:insert_block name="material"/>
-        </visual>
-    </xacro:macro>
+<robot xmlns:xacro="http://www.ros.org/wiki/xacro">
     <xacro:property name="robot_name" default="hdt_michigan"/>
     <xacro:property name="hardware_interface" default="hardware_interface/PositionJointInterface"/>
@@ -20,8 +9,5 @@
     <!-- constants -->
     <xacro:property name="M_PI" value="3.1415926535897931"/>
-    <!-- materials -->
-    <material name="black">
-        <color rgba="${0/255} ${0/255} ${0/255} 1.0"/>
-    </material>
+    <xacro:property name="CONTINUOUS_LIM" value="6.2"/>
     <material name="grey">
         <color rgba="${60/255} ${60/255} ${60/255} 1.0"/>
@@ -33,7 +19,4 @@
         <color rgba="${128/255} ${0/255} ${0/255} 1.0"/>
     </material>
-    <material name="white">
-        <color rgba="${255/255} ${255/255} ${255/255} 1.0"/>
-    </material>
     <material name="blue">
         <color rgba="${4/255} ${30/255} ${66/255} 1.0"/>
@@ -44,51 +27,11 @@
     <!-- import gazebo definitions -->
     <xacro:include filename="$(find hdt_michigan_description)/urdf/hdt_michigan.gazebo.xacro"/>
-    <!-- segment 0 -->
     <link name="${robot_name}_root"/>
-    <joint name="husky_joint" type="fixed">
-        <origin xyz="0 0 0" rpy="0 0 0"/>
-        <parent link="hdt_michigan_root"/>
-        <child link="husky"/>
-    </joint>
-    <link name="husky">
-        <inertial>
-            <origin xyz="0 -0.32 -0.25" rpy="0 0 0"/>
-            <mass value="25"/>
-            <inertia ixx="2.338"
-                     ixy="0"
-                     ixz="0"
-                     iyy="2.338"
-                     iyz="0"
-                     izz="4.166"/>
-        </inertial>
-        <xacro:collision_visual name="husky_base">
-            <!-- NOTE: the order of the following elements matters! -->
-            <origin xyz="0 -0.32 -0.15" rpy="0 0 0"/>
-            <geometry>
-                <box size="1 1 0.37"/>
-            </geometry>
-            <material name="black"/>
-        </xacro:collision_visual>
-        <xacro:collision_visual name="protect_cables">
-            <origin xyz="0.0 -0.1 0.18" rpy="0 0 0"/>
-            <geometry>
-                <box size="0.2 0.2 0.4"/>
-            </geometry>
-            <material name="maize"/>
-        </xacro:collision_visual>
-        <xacro:collision_visual name="battery">
-            <origin xyz="0 -0.50 0.10" rpy="0 0 0"/>
-            <geometry>
-                <box size="1 0.65 0.4"/>
-            </geometry>
-            <material name="maize"/>
-        </xacro:collision_visual>
-    </link>
+    <link name="base"/>
     <joint name="base" type="fixed">
         <origin xyz="0 0 0" rpy="0 0 0"/>
-        <parent link="hdt_michigan_root"/>
+        <parent link="${robot_name}_root"/>
         <child link="base"/>
     </joint>
-    <link name="base"/>
     <link name="realsense">
         <collision name="realsense_collision">
@@ -173,5 +116,5 @@
         <hdt id="56" kmin="100" kmax="200" inertia="0.1"/>
         <axis xyz="0 -1 0"/>
-        <limit effort="180.0" lower="${-2*M_PI}" upper="${2*M_PI}" velocity="0.45"/>
+        <limit effort="180.0" lower="${-CONTINUOUS_LIM}" upper="${CONTINUOUS_LIM}" velocity="0.45"/>
         <origin xyz="0 0 -.082642" rpy="${M_PI/2} 0 ${M_PI/2}"/>
         <parent link="drive56"/>
@@ -272,5 +215,5 @@
         <hdt id="41" kmin="100" kmax="200" inertia="0.1"/>
         <axis xyz="0 1 0"/>
-        <limit effort="18.0" lower="${-2*M_PI}" upper="${2*M_PI}" velocity="0.45"/>
+        <limit effort="180.0" lower="${-CONTINUOUS_LIM}" upper="${CONTINUOUS_LIM}" velocity="0.45"/>
         <origin xyz="0 0 -.082642" rpy="${M_PI/2} 0 -${M_PI/2}"/>
         <parent link="drive41"/>
@@ -369,5 +312,5 @@
         <hdt id="43" kmin="100" kmax="200" inertia="0.1"/>
         <axis xyz="0 0 -1"/>
-        <limit effort="90.0" lower="${-2*M_PI}" upper="${2*M_PI}" velocity="0.45"/>
+        <limit effort="90.0" lower="${-CONTINUOUS_LIM}" upper="${CONTINUOUS_LIM}" velocity="0.45"/>
         <origin xyz="0 0 -.115888" rpy="${-M_PI} 0 0"/>
         <parent link="drive43"/>
@@ -495,5 +438,5 @@
         <hdt id="45" kmin="100" kmax="200" inertia="0.1"/>
         <axis xyz="0 1 0"/>
-        <limit effort="35.0" lower="${-2*M_PI}" upper="${2*M_PI}" velocity="${2*M_PI/3}"/>
+        <limit effort="35.0" lower="${-CONTINUOUS_LIM}" upper="${CONTINUOUS_LIM}" velocity="${2*M_PI/3}"/>
         <origin xyz="0 0 -.067262" rpy="${M_PI/2} 0 ${M_PI/2}"/>
         <parent link="drive45"/>
@@ -592,5 +535,5 @@
         <hdt id="47" kmin="100" kmax="200" inertia="0.1"/>
         <axis xyz="0 0 -1"/>
-        <limit effort="35.0" lower="${-2*M_PI}" upper="${2*M_PI}" velocity="${M_PI}"/>
+        <limit effort="35.0" lower="${-CONTINUOUS_LIM}" upper="${CONTINUOUS_LIM}" velocity="${M_PI}"/>
         <origin xyz="0 0 -.036" rpy="${M_PI} 0 ${M_PI}"/>
         <parent link="drive47"/>
@@ -611,4 +554,10 @@
             <geometry>
                 <mesh filename="package://hdt_michigan_description/meshes/PINCER_HOUSING2.STL" scale="1.0 1.0 1.0"/>
+            </geometry>
+        </collision>
+        <collision>
+            <origin xyz="0.0625 0 0.045" rpy="0 0 0"/>
+            <geometry>
+                <box size="0.03 0.10 0.10"/>
             </geometry>
         </collision>
@@ -736,5 +685,5 @@
         <hdt id="1" kmin="100" kmax="200" inertia="0.1"/>
         <axis xyz="0 -1 0"/>
-        <limit effort="180.0" lower="${-2*M_PI}" upper="${2*M_PI}" velocity="0.45"/>
+        <limit effort="180.0" lower="${-CONTINUOUS_LIM}" upper="${CONTINUOUS_LIM}" velocity="0.45"/>
         <origin xyz="0 0 -.082642" rpy="${M_PI/2} 0 ${M_PI/2}"/>
         <parent link="drive1"/>
@@ -833,5 +782,5 @@
         <hdt id="3" kmin="100" kmax="200" inertia="0.1"/>
         <axis xyz="0 0 -1"/>
-        <limit effort="90.0" lower="${-2*M_PI}" upper="${2*M_PI}" velocity="0.45"/>
+        <limit effort="90.0" lower="${-CONTINUOUS_LIM}" upper="${CONTINUOUS_LIM}" velocity="0.45"/>
         <origin xyz="0 0 -.115888" rpy="${-M_PI} 0 ${M_PI}"/>
         <parent link="drive3"/>
@@ -959,5 +908,5 @@
         <hdt id="5" kmin="100" kmax="200" inertia="0.1"/>
         <axis xyz="0 1 0"/>
-        <limit effort="35.0" lower="${-2*M_PI}" upper="${2*M_PI}" velocity="${2*M_PI/3}"/>
+        <limit effort="35.0" lower="${-CONTINUOUS_LIM}" upper="${CONTINUOUS_LIM}" velocity="${2*M_PI/3}"/>
         <origin xyz="0 0 -.067262" rpy="${M_PI/2} 0 ${-M_PI/2}"/>
         <parent link="drive5"/>
@@ -1056,5 +1005,5 @@
         <hdt id="7" kmin="100" kmax="200" inertia="0.1"/>
         <axis xyz="0 0 -1"/>
-        <limit effort="35.0" lower="${-2*M_PI}" upper="${2*M_PI}" velocity="${M_PI}"/>
+        <limit effort="35.0" lower="${-CONTINUOUS_LIM}" upper="${CONTINUOUS_LIM}" velocity="${M_PI}"/>
         <origin xyz="0 0 -.036" rpy="${M_PI} 0 0"/>
         <parent link="drive7"/>
@@ -1075,4 +1024,10 @@
             <geometry>
                 <mesh filename="package://hdt_michigan_description/meshes/PINCER_HOUSING2.STL" scale="1.0 1.0 1.0"/>
+            </geometry>
+        </collision>
+        <collision>
+            <origin xyz="0.0625 0 0.045" rpy="0 0 0"/>
+            <geometry>
+                <box size="0.03 0.10 0.10"/>
             </geometry>
         </collision>
@@ -1219,4 +1174,3 @@
     <xacro:add_gazebo_control_plugin robot_namespace="${robot_name}"/>
     <xacro:add_moveit_planning_scene_plugin robot_namespace="${robot_name}" root_frame_id="${robot_name}_root"/>
-    <xacro:add_gazebo_fixed_link base_link="${robot_name}_root"/>
 </robot>

File: models/husky_custom_description/urdf/mic09_description.urdf (robot description, URDF)
Before this commit: robot hdt_michigan, 44 links, 43 joints
Links:
- removed link husky
- removed link left_hand
- removed link right_hand
- removed link val_cal
- removed link world
- added link base_footprint
- added link base_link; collision box size=0.7899200000000001 0.5709 0.10375; collision box size=0.9874 0.5709 0.12375
- added link front_bumper_link; visual mesh filename=package://husky_description/meshes/bumper.dae
- added link front_laser
- added link front_left_wheel_link, mass 2.637; collision cylinder length=0.1143 radius=0.1651; visual mesh filename=package://husky_description/meshes/wheel.dae
- added link front_lidar_mesh; collision mesh filename=package://husky_custom_description/meshes/ark_lidar.stl; visual mesh filename=package://husky_custom_description/meshes/ark_lidar.stl
- added link front_right_wheel_link, mass 2.637; collision cylinder length=0.1143 radius=0.1651; visual mesh filename=package://husky_description/meshes/wheel.dae
- added link imu_link
- added link inertial_link, mass 46.034
- added link rear_bumper_link; visual mesh filename=package://husky_description/meshes/bumper.dae
- added link rear_laser
- added link rear_left_wheel_link, mass 2.637; collision cylinder length=0.1143 radius=0.1651; visual mesh filename=package://husky_description/meshes/wheel.dae
- added link rear_lidar_mesh; collision mesh filename=package://husky_custom_description/meshes/ark_lidar.stl; visual mesh filename=package://husky_custom_description/meshes/ark_lidar.stl
- added link rear_right_wheel_link, mass 2.637; collision cylinder length=0.1143 radius=0.1651; visual mesh filename=package://husky_description/meshes/wheel.dae
- added link robot_payload; collision box size=.19 .18 .25; collision box size=.19 .18 .25
- added link robot_root
- added link top_chassis_link; visual mesh filename=package://husky_description/meshes/top_chassis.dae
- added link top_plate_front_link
- added link top_plate_link; collision mesh filename=package://husky_description/meshes/top_plate.stl; visual mesh filename=package://husky_description/meshes/top_plate.dae
- added link top_plate_rear_link
- added link user_rail_link; visual mesh filename=package://husky_description/meshes/user_rail.dae
- link end_effector_left: geometry collision box size=0.03 0.10 0.10; collision mesh filename=package://hdt_michigan_description/meshes/PINCER_HOUSING2.S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 scale=1.0 1.0 1.0
- link end_effector_right: geometry collision box size=0.03 0.10 0.10; collision mesh filename=package://hdt_michigan_description/meshes/PINCER_HOUSING2.S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 scale=1.0 1.0 1.0
- link leftgripper2_link: geometry collision mesh filename=package://hdt_michigan_description/meshes/PINCER_FINGER.STL scale=1.0 1.0 1.0; visual mesh filename=package://hdt_michigan_description/meshes/PINCER_FINGER.STL
- link leftgripper_link: geometry collision mesh filename=package://hdt_michigan_description/meshes/PINCER_FINGER.STL scale=1.0 1.0 1.0; visual mesh filename=package://hdt_michigan_description/meshes/PINCER_FINGER.STL
- link rightgripper2_link: geometry collision mesh filename=package://hdt_michigan_description/meshes/PINCER_FINGER.STL scale=1.0 1.0 1.0; visual mesh filename=package://hdt_michigan_description/meshes/PINCER_FINGER.STL
Joints:
- removed joint husky_joint
- removed joint left_hand_joint
- removed joint right_hand_joint
- removed joint val_cal_joint
- removed joint world_joint
- added joint base_footprint_joint: type fixed, parent base_link, child base_footprint, origin xyz=0 0 -0.13228 rpy=0 0 0
- added joint base_link_to_front_laser: type fixed, parent base_link, child front_laser, origin xyz=0.46 0.0 -0.04 rpy=0 0 0
- added joint base_link_to_front_lidar: type fixed, parent base_link, child front_lidar_mesh, origin xyz=0.412 0 0.068 rpy=0 0 0
- added joint base_link_to_hdt_michigan_root: type fixed, parent base_link, child hdt_michigan_root, origin xyz=0.275 -0.0047 0.335 rpy=-0.035 0 -1.5707
- added joint base_link_to_rear_laser: type fixed, parent base_link, child rear_laser, origin xyz=-0.46 0.0 -0.04 rpy=0 0 3.14159
- added joint base_link_to_rear_lidar: type fixed, parent base_link, child rear_lidar_mesh, origin xyz=-0.412 0 0.068 rpy=0 0 3.14159
- added joint front_bumper: type fixed, parent base_link, child front_bumper_link, origin xyz=0.48 0 0.091 rpy=0 0 0
- added joint front_left_wheel: type continuous, parent base_link, child front_left_wheel_link, origin xyz=0.256 0.2854 0.03282 rpy=0 0 0, axis 0 1 0
- added joint front_right_wheel: type continuous, parent base_link, child front_right_wheel_link, origin xyz=0.256 -0.2854 0.03282 rpy=0 0 0, axis 0 1 0
- added joint imu_joint: type fixed, parent base_link, child imu_link, origin xyz=0.19 0 0.149 rpy=0 -1.5708 3.1416
- added joint inertial_joint: type fixed, parent base_link, child inertial_link, origin xyz=0 0 0 rpy=0 0 0
- added joint rear_bumper: type fixed, parent base_link, child rear_bumper_link, origin xyz=-0.48 0 0.091 rpy=0 0 3.14159
- added joint rear_left_wheel: type continuous, parent base_link, child rear_left_wheel_link, origin xyz=-0.256 0.2854 0.03282 rpy=0 0 0, axis 0 1 0
- added joint rear_right_wheel: type continuous, parent base_link, child rear_right_wheel_link, origin xyz=-0.256 -0.2854 0.03282 rpy=0 0 0, axis 0 1 0
- added joint robot_payload_joint: type fixed, parent base_link, child robot_payload, origin xyz=0 0 0.35 rpy=0 0 0
- added joint robot_root_joint: type fixed, parent base_link, child robot_root, origin xyz=0 0 0 rpy=0 0 0
- added joint top_chassis_joint: type fixed, parent base_link, child top_chassis_link
- added joint top_plate_front_joint: type fixed, parent top_plate_link, child top_plate_front_link, origin xyz=0.36367 0 0.00639 rpy=0 0 0
- added joint top_plate_joint: type fixed, parent base_link, child top_plate_link, origin xyz=0.0812 0 0.245 rpy=0 0 0
- added joint top_plate_rear_joint: type fixed, parent top_plate_link, child top_plate_rear_link, origin xyz=-0.36633 0 0.00639 rpy=0 0 0
- added joint user_rail: type fixed, parent base_link, child user_rail_link, origin xyz=0.272 0 0.245 rpy=0 0 0
- joint joint1: limit lower=-6.283185307179586 upper=6.283185307179586 effort=180.0 velocity=0.45 -> lower=-6.2 upper=6.2 effort=180.0 velocity=0.45
- joint joint3: limit lower=-6.283185307179586 upper=6.283185307179586 effort=90.0 velocity=0.45 -> lower=-6.2 upper=6.2 effort=90.0 velocity=0.45
- joint joint41: limit lower=-6.283185307179586 upper=6.283185307179586 effort=18.0 velocity=0.45 -> lower=-6.2 upper=6.2 effort=180.0 velocity=0.45
- joint joint43: limit lower=-6.283185307179586 upper=6.283185307179586 effort=90.0 velocity=0.45 -> lower=-6.2 upper=6.2 effort=90.0 velocity=0.45
- joint joint45: limit lower=-6.283185307179586 upper=6.283185307179586 effort=35.0 velocity=2.0943951023931953 -> lower=-6.2 upper=6.2 effort=35.0 velocity=2.0943951023931953
- joint joint47: limit lower=-6.283185307179586 upper=6.283185307179586 effort=35.0 velocity=3.141592653589793 -> lower=-6.2 upper=6.2 effort=35.0 velocity=3.141592653589793
- joint joint5: limit lower=-6.283185307179586 upper=6.283185307179586 effort=35.0 velocity=2.0943951023931953 -> lower=-6.2 upper=6.2 effort=35.0 velocity=2.0943951023931953
- joint joint56: limit lower=-6.283185307179586 upper=6.283185307179586 effort=180.0 velocity=0.45 -> lower=-6.2 upper=6.2 effort=180.0 velocity=0.45
- joint joint7: limit lower=-6.283185307179586 upper=6.283185307179586 effort=35.0 velocity=3.141592653589793 -> lower=-6.2 upper=6.2 effort=35.0 velocity=3.141592653589793
