Commit message: new URDF

File: models/victor_description/urdf/victor.urdf (robot description, URDF)
Before this commit: robot victor, 60 links, 59 joints
Links:
- removed link victor_left_gripper_fingerA_base
- removed link victor_left_gripper_fingerA_dist
- removed link victor_left_gripper_fingerA_med
- removed link victor_left_gripper_fingerA_prox
- removed link victor_left_gripper_fingerB_base
- removed link victor_left_gripper_fingerB_dist
- removed link victor_left_gripper_fingerB_med
- removed link victor_left_gripper_fingerB_prox
- removed link victor_left_gripper_fingerC_base
- removed link victor_left_gripper_fingerC_dist
- removed link victor_left_gripper_fingerC_med
- removed link victor_left_gripper_fingerC_prox
- removed link victor_left_gripper_palm
- removed link victor_left_gripper_palm_surface
- removed link victor_left_gripper_palm_surface_kuka
- removed link victor_right_gripper_fingerA_base
- removed link victor_right_gripper_fingerA_dist
- removed link victor_right_gripper_fingerA_med
- removed link victor_right_gripper_fingerA_prox
- removed link victor_right_gripper_fingerB_base
- removed link victor_right_gripper_fingerB_dist
- removed link victor_right_gripper_fingerB_med
- removed link victor_right_gripper_fingerB_prox
- removed link victor_right_gripper_fingerC_base
- removed link victor_right_gripper_fingerC_dist
- removed link victor_right_gripper_fingerC_med
- removed link victor_right_gripper_fingerC_prox
- removed link victor_right_gripper_palm
- removed link victor_right_gripper_palm_surface
- removed link victor_right_gripper_palm_surface_kuka
- added link l_finger_1_link_0, mass 0.1; collision mesh filename=package://robotiq_3f_gripper_visualization/meshes/robotiq-3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; visual mesh filename=package://robotiq_3f_gripper_visualization/meshes/robotiq-3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
- added link l_finger_1_link_1, mass 0.047; collision mesh filename=package://robotiq_3f_gripper_visualization/meshes/robotiq-3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; visual mesh filename=package://robotiq_3f_gripper_visualization/meshes/robotiq-3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
- added link l_finger_1_link_2, mass 0.03284; collision mesh filename=package://robotiq_3f_gripper_visualization/meshes/robotiq-3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; visual mesh filename=package://robotiq_3f_gripper_visualization/meshes/robotiq-3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
- added link l_finger_1_link_3, mass 0.03354; collision mesh filename=package://robotiq_3f_gripper_visualization/meshes/robotiq-3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; visual mesh filename=package://robotiq_3f_gripper_visualization/meshes/robotiq-3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
- added link l_finger_2_link_0, mass 0.1; collision mesh filename=package://robotiq_3f_gripper_visualization/meshes/robotiq-3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; visual mesh filename=package://robotiq_3f_gripper_visualization/meshes/robotiq-3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
- added link l_finger_2_link_1, mass 0.047; collision mesh filename=package://robotiq_3f_gripper_visualization/meshes/robotiq-3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; visual mesh filename=package://robotiq_3f_gripper_visualization/meshes/robotiq-3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
- added link l_finger_2_link_2, mass 0.03284; collision mesh filename=package://robotiq_3f_gripper_visualization/meshes/robotiq-3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; visual mesh filename=package://robotiq_3f_gripper_visualization/meshes/robotiq-3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
- added link l_finger_2_link_3, mass 0.03354; collision mesh filename=package://robotiq_3f_gripper_visualization/meshes/robotiq-3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; visual mesh filename=package://robotiq_3f_gripper_visualization/meshes/robotiq-3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
- added link l_finger_middle_link_0, mass 0.1; collision mesh filename=package://robotiq_3f_gripper_visualization/meshes/robotiq-3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; visual mesh filename=package://robotiq_3f_gripper_visualization/meshes/robotiq-3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
- added link l_finger_middle_link_1, mass 0.047; collision mesh filename=package://robotiq_3f_gripper_visualization/meshes/robotiq-3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; visual mesh filename=package://robotiq_3f_gripper_visualization/meshes/robotiq-3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
- added link l_finger_middle_link_2, mass 0.03284; collision mesh filename=package://robotiq_3f_gripper_visualization/meshes/robotiq-3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; visual mesh filename=package://robotiq_3f_gripper_visualization/meshes/robotiq-3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
- added link l_finger_middle_link_3, mass 0.03354; collision mesh filename=package://robotiq_3f_gripper_visualization/meshes/robotiq-3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; visual mesh filename=package://robotiq_3f_gripper_visualization/meshes/robotiq-3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
- added link l_palm, mass 1.3; collision box size=0.1 0.1 0.1; visual mesh filename=package://robotiq_3f_gripper_visualization/meshes/robotiq-3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
- added link left_tool, mass 0.001; visual sphere radius=0.002
- added link r_finger_1_link_0, mass 0.1; collision mesh filename=package://robotiq_3f_gripper_visualization/meshes/robotiq-3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; visual mesh filename=package://robotiq_3f_gripper_visualization/meshes/robotiq-3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
- added link r_finger_1_link_1, mass 0.047; collision mesh filename=package://robotiq_3f_gripper_visualization/meshes/robotiq-3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; visual mesh filename=package://robotiq_3f_gripper_visualization/meshes/robotiq-3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
- added link r_finger_1_link_2, mass 0.03284; collision mesh filename=package://robotiq_3f_gripper_visualization/meshes/robotiq-3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; visual mesh filename=package://robotiq_3f_gripper_visualization/meshes/robotiq-3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
- added link r_finger_1_link_3, mass 0.03354; collision mesh filename=package://robotiq_3f_gripper_visualization/meshes/robotiq-3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; visual mesh filename=package://robotiq_3f_gripper_visualization/meshes/robotiq-3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
- added link r_finger_2_link_0, mass 0.1; collision mesh filename=package://robotiq_3f_gripper_visualization/meshes/robotiq-3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; visual mesh filename=package://robotiq_3f_gripper_visualization/meshes/robotiq-3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
- added link r_finger_2_link_1, mass 0.047; collision mesh filename=package://robotiq_3f_gripper_visualization/meshes/robotiq-3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; visual mesh filename=package://robotiq_3f_gripper_visualization/meshes/robotiq-3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
- added link r_finger_2_link_2, mass 0.03284; collision mesh filename=package://robotiq_3f_gripper_visualization/meshes/robotiq-3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; visual mesh filename=package://robotiq_3f_gripper_visualization/meshes/robotiq-3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
- added link r_finger_2_link_3, mass 0.03354; collision mesh filename=package://robotiq_3f_gripper_visualization/meshes/robotiq-3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; visual mesh filename=package://robotiq_3f_gripper_visualization/meshes/robotiq-3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
- added link r_finger_middle_link_0, mass 0.1; collision mesh filename=package://robotiq_3f_gripper_visualization/meshes/robotiq-3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; visual mesh filename=package://robotiq_3f_gripper_visualization/meshes/robotiq-3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
- added link r_finger_middle_link_1, mass 0.047; collision mesh filename=package://robotiq_3f_gripper_visualization/meshes/robotiq-3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; visual mesh filename=package://robotiq_3f_gripper_visualization/meshes/robotiq-3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
- added link r_finger_middle_link_2, mass 0.03284; collision mesh filename=package://robotiq_3f_gripper_visualization/meshes/robotiq-3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; visual mesh filename=package://robotiq_3f_gripper_visualization/meshes/robotiq-3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
- added link r_finger_middle_link_3, mass 0.03354; collision mesh filename=package://robotiq_3f_gripper_visualization/meshes/robotiq-3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; visual mesh filename=package://robotiq_3f_gripper_visualization/meshes/robotiq-3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
- added link r_palm, mass 1.3; collision box size=0.1 0.1 0.1; visual mesh filename=package://robotiq_3f_gripper_visualization/meshes/robotiq-3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
- added link right_tool, mass 0.001; visual sphere radius=0.002
- added link world
Joints:
- removed joint victor_left_gripper_fingerA_joint_2
- removed joint victor_left_gripper_fingerA_joint_3
- removed joint victor_left_gripper_fingerA_joint_4
- removed joint victor_left_gripper_fingerA_knuckle
- removed joint victor_left_gripper_fingerB_joint_2
- removed joint victor_left_gripper_fingerB_joint_3
- removed joint victor_left_gripper_fingerB_joint_4
- removed joint victor_left_gripper_fingerB_knuckle
- removed joint victor_left_gripper_fingerC_joint_2
- removed joint victor_left_gripper_fingerC_joint_3
- removed joint victor_left_gripper_fingerC_joint_4
- removed joint victor_left_gripper_fingerC_knuckle
- removed joint victor_left_gripper_palm_joint
- removed joint victor_left_gripper_palm_surface_joint
- removed joint victor_left_gripper_palm_surface_kuka_joint
- removed joint victor_right_gripper_fingerA_joint_2
- removed joint victor_right_gripper_fingerA_joint_3
- removed joint victor_right_gripper_fingerA_joint_4
- removed joint victor_right_gripper_fingerA_knuckle
- removed joint victor_right_gripper_fingerB_joint_2
- removed joint victor_right_gripper_fingerB_joint_3
- removed joint victor_right_gripper_fingerB_joint_4
- removed joint victor_right_gripper_fingerB_knuckle
- removed joint victor_right_gripper_fingerC_joint_2
- removed joint victor_right_gripper_fingerC_joint_3
- removed joint victor_right_gripper_fingerC_joint_4
- removed joint victor_right_gripper_fingerC_knuckle
- removed joint victor_right_gripper_palm_joint
- removed joint victor_right_gripper_palm_surface_joint
- removed joint victor_right_gripper_palm_surface_kuka_joint
- added joint l_finger_1_joint_1: type revolute, parent l_finger_1_link_0, child l_finger_1_link_1, origin xyz=0 0 0 rpy=0 0 -2.0906, axis 0 0 1, limit lower=0 upper=1.2217 effort=60 velocity=-1
- added joint l_finger_1_joint_2: type revolute, parent l_finger_1_link_1, child l_finger_1_link_2, origin xyz=0 0.05715 0 rpy=0 0 0, axis 0 0 1, limit lower=0 upper=1.5708 effort=60 velocity=-1
- added joint l_finger_1_joint_3: type revolute, parent l_finger_1_link_2, child l_finger_1_link_3, origin xyz=0 0.039 0 rpy=0 0 2.0906000000000002, axis 0 0 1, limit lower=-0.6632 upper=1.0471 effort=60 velocity=-1
- added joint l_finger_2_joint_1: type revolute, parent l_finger_2_link_0, child l_finger_2_link_1, origin xyz=0 0 0 rpy=0 0 -2.0906, axis 0 0 1, limit lower=0 upper=1.2217 effort=60 velocity=-1
- added joint l_finger_2_joint_2: type revolute, parent l_finger_2_link_1, child l_finger_2_link_2, origin xyz=0 0.05715 0 rpy=0 0 0, axis 0 0 1, limit lower=0 upper=1.5708 effort=60 velocity=-1
- added joint l_finger_2_joint_3: type revolute, parent l_finger_2_link_2, child l_finger_2_link_3, origin xyz=0 0.039 0 rpy=0 0 2.0906000000000002, axis 0 0 1, limit lower=-0.6632 upper=1.0471 effort=60 velocity=-1
- added joint l_finger_middle_joint_1: type revolute, parent l_finger_middle_link_0, child l_finger_middle_link_1, origin xyz=0 0 0 rpy=0 0 -2.0906, axis 0 0 1, limit lower=0 upper=1.2217 effort=60 velocity=-1
- added joint l_finger_middle_joint_2: type revolute, parent l_finger_middle_link_1, child l_finger_middle_link_2, origin xyz=0 0.05715 0 rpy=0 0 0, axis 0 0 1, limit lower=0 upper=1.5708 effort=60 velocity=-1
- added joint l_finger_middle_joint_3: type revolute, parent l_finger_middle_link_2, child l_finger_middle_link_3, origin xyz=0 0.039 0 rpy=0 0 2.0906000000000002, axis 0 0 1, limit lower=-0.6632 upper=1.0471 effort=60 velocity=-1
- added joint l_palm_finger_1_joint: type revolute, parent l_palm, child l_finger_1_link_0, origin xyz=-0.0455 0.0214 0.036 rpy=0 3.1416 -1.57, axis 0 1 0, limit lower=-0.2967 upper=0.2967 effort=60 velocity=-1
- added joint l_palm_finger_2_joint: type revolute, parent l_palm, child l_finger_2_link_0, origin xyz=-0.0455 0.0214 -0.036 rpy=0 3.1416 -1.57, axis 0 1 0, limit lower=-0.2967 upper=0.2967 effort=60 velocity=-1
- added joint l_palm_finger_middle_joint: type fixed, parent l_palm, child l_finger_middle_link_0, origin xyz=0.0455 0.0214 0 rpy=0 0 1.57, axis 0 1 0, limit lower=0 upper=0 effort=60 velocity=-1
- added joint l_robotiq_hand_joint: type fixed, parent victor_left_gripper_mounting_bracket, child l_palm, origin xyz=0 0 0.07 rpy=1.5707963267948966 0 0.7853981633974483
- added joint left_tool_joint: type fixed, parent victor_left_arm_link_7, child left_tool, origin xyz=0 0 0.254
- added joint r_finger_1_joint_1: type revolute, parent r_finger_1_link_0, child r_finger_1_link_1, origin xyz=0 0 0 rpy=0 0 -2.0906, axis 0 0 1, limit lower=0 upper=1.2217 effort=60 velocity=-1
- added joint r_finger_1_joint_2: type revolute, parent r_finger_1_link_1, child r_finger_1_link_2, origin xyz=0 0.05715 0 rpy=0 0 0, axis 0 0 1, limit lower=0 upper=1.5708 effort=60 velocity=-1
- added joint r_finger_1_joint_3: type revolute, parent r_finger_1_link_2, child r_finger_1_link_3, origin xyz=0 0.039 0 rpy=0 0 2.0906000000000002, axis 0 0 1, limit lower=-0.6632 upper=1.0471 effort=60 velocity=-1
- added joint r_finger_2_joint_1: type revolute, parent r_finger_2_link_0, child r_finger_2_link_1, origin xyz=0 0 0 rpy=0 0 -2.0906, axis 0 0 1, limit lower=0 upper=1.2217 effort=60 velocity=-1
- added joint r_finger_2_joint_2: type revolute, parent r_finger_2_link_1, child r_finger_2_link_2, origin xyz=0 0.05715 0 rpy=0 0 0, axis 0 0 1, limit lower=0 upper=1.5708 effort=60 velocity=-1
- added joint r_finger_2_joint_3: type revolute, parent r_finger_2_link_2, child r_finger_2_link_3, origin xyz=0 0.039 0 rpy=0 0 2.0906000000000002, axis 0 0 1, limit lower=-0.6632 upper=1.0471 effort=60 velocity=-1
- added joint r_finger_middle_joint_1: type revolute, parent r_finger_middle_link_0, child r_finger_middle_link_1, origin xyz=0 0 0 rpy=0 0 -2.0906, axis 0 0 1, limit lower=0 upper=1.2217 effort=60 velocity=-1
- added joint r_finger_middle_joint_2: type revolute, parent r_finger_middle_link_1, child r_finger_middle_link_2, origin xyz=0 0.05715 0 rpy=0 0 0, axis 0 0 1, limit lower=0 upper=1.5708 effort=60 velocity=-1
- added joint r_finger_middle_joint_3: type revolute, parent r_finger_middle_link_2, child r_finger_middle_link_3, origin xyz=0 0.039 0 rpy=0 0 2.0906000000000002, axis 0 0 1, limit lower=-0.6632 upper=1.0471 effort=60 velocity=-1
- added joint r_palm_finger_1_joint: type revolute, parent r_palm, child r_finger_1_link_0, origin xyz=-0.0455 0.0214 0.036 rpy=0 3.1416 -1.57, axis 0 1 0, limit lower=-0.2967 upper=0.2967 effort=60 velocity=-1
- added joint r_palm_finger_2_joint: type revolute, parent r_palm, child r_finger_2_link_0, origin xyz=-0.0455 0.0214 -0.036 rpy=0 3.1416 -1.57, axis 0 1 0, limit lower=-0.2967 upper=0.2967 effort=60 velocity=-1
- added joint r_palm_finger_middle_joint: type fixed, parent r_palm, child r_finger_middle_link_0, origin xyz=0.0455 0.0214 0 rpy=0 0 1.57, axis 0 1 0, limit lower=0 upper=0 effort=60 velocity=-1
- added joint r_robotiq_hand_joint: type fixed, parent victor_right_gripper_mounting_bracket, child r_palm, origin xyz=0 0 0.07 rpy=1.5707963267948966 0 0.7853981633974483
- added joint right_tool_joint: type fixed, parent victor_right_arm_link_7, child right_tool, origin xyz=0 0 0.254
- added joint world_joint: type fixed, parent world, child victor_root, origin xyz=0.0 0.0 0.0 rpy=0.0 0.0 0.0
- joint victor_left_arm_flange_victor_left_joint: origin xyz=0 0 0 rpy=0 0 0 -> xyz=0 0 -0.01 rpy=0 0 0
- joint victor_left_arm_joint_1: limit lower=-2.96705972839 upper=2.96705972839 effort=300 velocity=10 -> lower=-2.9670597283903604 upper=2.9670597283903604 effort=300 velocity=1.7453292519943295
- joint victor_left_arm_joint_2: limit lower=-2.09439510239 upper=2.09439510239 effort=300 velocity=10 -> lower=-2.0943951023931953 upper=2.0943951023931953 effort=300 velocity=1.7453292519943295; origin xyz=0 0 0.19 rpy=1.57079632679   0 3.14159265359 -> xyz=0 0 0.19 rpy=1.5707963267948966   0 3.141592653589793
- joint victor_left_arm_joint_3: limit lower=-2.96705972839 upper=2.96705972839 effort=300 velocity=10 -> lower=-2.9670597283903604 upper=2.9670597283903604 effort=300 velocity=1.7453292519943295; origin xyz=0 0.21 0 rpy=1.57079632679 0 3.14159265359 -> xyz=0 0.21 0 rpy=1.5707963267948966 0 3.141592653589793
- joint victor_left_arm_joint_4: limit lower=-2.09439510239 upper=2.09439510239 effort=300 velocity=10 -> lower=-2.0943951023931953 upper=2.0943951023931953 effort=300 velocity=2.2689280275926285; origin xyz=0 0 0.19 rpy=1.57079632679 0 0 -> xyz=0 0 0.19 rpy=1.5707963267948966 0 0
- joint victor_left_arm_joint_5: limit lower=-2.96705972839 upper=2.96705972839 effort=300 velocity=10 -> lower=-2.9670597283903604 upper=2.9670597283903604 effort=300 velocity=2.443460952792061; origin xyz=0 0.21 0 rpy=-1.57079632679 3.14159265359 0 -> xyz=0 0.21 0 rpy=-1.5707963267948966 3.141592653589793 0
- joint victor_left_arm_joint_6: limit lower=-2.09439510239 upper=2.09439510239 effort=300 velocity=10 -> lower=-2.0943951023931953 upper=2.0943951023931953 effort=300 velocity=3.141592653589793; origin xyz=0 0.06070 0.19 rpy=1.57079632679 0 0 -> xyz=0 0.06070 0.19 rpy=1.5707963267948966 0 0
- joint victor_left_arm_joint_7: limit lower=-3.05432619099 upper=3.05432619099 effort=300 velocity=10 -> lower=-3.0543261909900763 upper=3.0543261909900763 effort=300 velocity=3.141592653589793; origin xyz=0 0.081 0.06070 rpy=-1.57079632679 3.14159265359 0 -> xyz=0 0.081 0.06070 rpy=-1.5707963267948966 3.141592653589793 0
- joint victor_right_arm_flange_victor_right_joint: origin xyz=0 0 0 rpy=0 0 0 -> xyz=0 0 -0.01 rpy=0 0 0
- joint victor_right_arm_joint_1: limit lower=-2.96705972839 upper=2.96705972839 effort=300 velocity=10 -> lower=-2.9670597283903604 upper=2.9670597283903604 effort=300 velocity=1.7453292519943295
- joint victor_right_arm_joint_2: limit lower=-2.09439510239 upper=2.09439510239 effort=300 velocity=10 -> lower=-2.0943951023931953 upper=2.0943951023931953 effort=300 velocity=1.7453292519943295; origin xyz=0 0 0.19 rpy=1.57079632679   0 3.14159265359 -> xyz=0 0 0.19 rpy=1.5707963267948966   0 3.141592653589793
- joint victor_right_arm_joint_3: limit lower=-2.96705972839 upper=2.96705972839 effort=300 velocity=10 -> lower=-2.9670597283903604 upper=2.9670597283903604 effort=300 velocity=1.7453292519943295; origin xyz=0 0.21 0 rpy=1.57079632679 0 3.14159265359 -> xyz=0 0.21 0 rpy=1.5707963267948966 0 3.141592653589793
- joint victor_right_arm_joint_4: limit lower=-2.09439510239 upper=2.09439510239 effort=300 velocity=10 -> lower=-2.0943951023931953 upper=2.0943951023931953 effort=300 velocity=2.2689280275926285; origin xyz=0 0 0.19 rpy=1.57079632679 0 0 -> xyz=0 0 0.19 rpy=1.5707963267948966 0 0
- joint victor_right_arm_joint_5: limit lower=-2.96705972839 upper=2.96705972839 effort=300 velocity=10 -> lower=-2.9670597283903604 upper=2.9670597283903604 effort=300 velocity=2.443460952792061; origin xyz=0 0.21 0 rpy=-1.57079632679 3.14159265359 0 -> xyz=0 0.21 0 rpy=-1.5707963267948966 3.141592653589793 0
- joint victor_right_arm_joint_6: limit lower=-2.09439510239 upper=2.09439510239 effort=300 velocity=10 -> lower=-2.0943951023931953 upper=2.0943951023931953 effort=300 velocity=3.141592653589793; origin xyz=0 0.06070 0.19 rpy=1.57079632679 0 0 -> xyz=0 0.06070 0.19 rpy=1.5707963267948966 0 0
- joint victor_right_arm_joint_7: limit lower=-3.05432619099 upper=3.05432619099 effort=300 velocity=10 -> lower=-3.0543261909900763 upper=3.0543261909900763 effort=300 velocity=3.141592653589793; origin xyz=0 0.081 0.06070 rpy=-1.57079632679 3.14159265359 0 -> xyz=0 0.081 0.06070 rpy=-1.5707963267948966 3.141592653589793 0
