Commit message: new link for ar tag

File: models/husky_custom_description/urdf/mic09_description.urdf (robot description, URDF)
Before this commit: robot husky, 60 links, 59 joints
Links:
- added link ar_link, mass 0.27265869; collision box size=0.03 0.10 0.10; collision mesh filename=package://hdt_michigan_description/meshes/AR_TAG.obj scale=1.0 1.0 1.0
- link end_effector_left: geometry collision box size=0.03 0.10 0.10; collision mesh filename=package://hdt_michigan_description/meshes/PINCER_HOUSING2.S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 scale=1.0 1.0 1.0
Joints:
- added joint ar_joint: type fixed, parent end_effector_left, child ar_link, origin xyz=0 0 0 rpy=0 0 0

Commit message: camera link

File: models/husky_custom_description/urdf/mic09_description.urdf (robot description, URDF)
Before this commit: robot husky, 61 links, 60 joints
Links:
- added link cam, mass 0.27265869; collision box size=0.03 0.10 0.10; visual box size=0.03 0.10 0.10
Joints:
- added joint torso_to_cam: type fixed, parent torso, child cam, origin xyz=0 0 .44399 rpy=-1.570796 0 0
